File: tlc555cp_christmas/tlc555cp_christmas.kicad_sch (KiCad schematic)
At the start: 18 parts, among them SW1 SW_MEC_5E, U1 TLC555xP

Commit message: versior ordered on january 8 2023
Parts:
- C2: value 100u -> 3.3u
- R3: value 220k -> 10M
Other:
- note added: "t=RC=(10Mohm)(3.3uF) = 33s"
- note removed: "300s = R(100uF) -> R = 300/(100uF) = 3MOhms"
- note removed: "30s = RC -> C = 30s/R = 30s/4700 ohms = 6.4mF Do again C = 30s/100000ohms = .3mF"
- note removed: "use the 1Mohm for now"
Changed lines of the file:
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@@
     (stroke (width 0) (type default) (color 0 0 0 0))
   )
-  (text "300s = R(100uF) -> R = 300/(100uF) = 3MOhms" (at 198.12 92.71 0)
+  (text "t=RC=(10Mohm)(3.3uF) = 33s" (at 191.77 85.09 0)
     (effects (font (size 1.27 1.27)) (justify left bottom))
   )
-  (text "use the 1Mohm for now" (at 196.85 68.58 0)
-    (effects (font (size 1.27 1.27)) (justify left bottom))
-  )
   (text "V=IR\nV=Vcc - Vled = 3V - 2V = 1V\nR=V/I = 1V/10mA = 100ohms\n\nI and Vled are take from this\nparticular LED: https://www.digikey.ca/en/products/detail/sunled/XLUG11D/4745837\n\nUse 220 ohm values for now."
-    (at 101.6 149.86 0)
-    (effects (font (size 1.27 1.27)) (justify left bottom))
-  )
-  (text "30s = RC -> C = 30s/R = 30s/4700 ohms = 6.4mF\nDo again\nC = 30s/100000ohms = .3mF"
-    (at 196.85 87.63 0)
+    (at 88.9 151.13 0)
     (effects (font (size 1.27 1.27)) (justify left bottom))
   )
@@
       (effects (font (size 1.27 1.27)) (justify left))
     )
-    (property "Value" "100u" (id 1) (at 191.77 96.9009 0)
+    (property "Value" "3.3u" (id 1) (at 191.77 96.9009 0)
       (effects (font (size 1.27 1.27)) (justify left))
     )
@@
       (effects (font (size 1.27 1.27)) (justify left))
     )
-    (property "Value" "220k" (id 1) (at 190.5 68.5799 0)
+    (property "Value" "10M" (id 1) (at 190.5 68.5799 0)
       (effects (font (size 1.27 1.27)) (justify left))
     )
@@
     )
     (path "/04de272d-6ab3-4595-b8f1-32ad84c01e5f"
-      (reference "C2") (unit 1) (value "100u") (footprint "Capacitor_THT:CP_Radial_D5.0mm_P2.50mm")
+      (reference "C2") (unit 1) (value "3.3u") (footprint "Capacitor_THT:CP_Radial_D5.0mm_P2.50mm")
     )
     (path "/ec7b9779-5c2e-4e86-88dc-be53252ebba9"
@@
     )
     (path "/f821fc82-b807-4424-94d1-4d16b48aac1e"
-      (reference "R3") (unit 1) (value "220k") (footprint "Resistor_THT:R_Axial_DIN0204_L3.6mm_D1.6mm_P5.08mm_Horizontal")
+      (reference "R3") (unit 1) (value "10M") (footprint "Resistor_THT:R_Axial_DIN0204_L3.6mm_D1.6mm_P5.08mm_Horizontal")
     )
     (path "/27556d9f-cb64-4ecd-a410-d95fd8374a03"
