File: tlc555cp_easter/tlc555cp_easter.kicad_sch (KiCad schematic)
At the start: 18 parts, among them SW1 SW_MEC_5E, U1 TLC555xP

Commit message: Fix switch footprint pad assignment.
Parts:
- removed C1: 0.1u, Capacitor_THT:CP_Radial_D4.0mm_P2.00mm, symbol Device:C_Polarized
- added C1: 0.1U, Capacitor_THT:CP_Radial_D5.0mm_P2.50mm, symbol Device:C
Connections:
- net GND: now also C1.2
- net at U1.5 (CV): now also C1.1
Other:
- note added: "Let's figure the approximate LED current. Vcc = 6V (will be a bit less) Vpled = forward voltage of the purple LED = 3.2V Vrled = forward voltage of the red LED = 2V Voled = forward voltage of the orange LED = 2V R = 220 Ohm Irled = Ioled V=Vcc - Vrled=IR Irled = 4V/220 Ohm = 18mA Ipled = 13 mA There may be rounding errors in these calculations but they should be fairly close. This means that the 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"
- note added: "Lets figure the off current. The 10M Ohm resistor will have a current draw. Vcc=IR -> 6V=I (10M Ohm) -> I = 6V/(10M Ohm) = 0.6uA (micro-amps!) Not very much there! On page one of the data sheet we see P=1mW at Vdd = 5V lets figure out the current consumption: P=VI -> I = P/V -> I = 1mW/5V = 0.2mA. So that is more significant! Plus our batteries discharge about 1% a year by themselves (see energiz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"
- note added: "Pin 2 is pulled high with a current limiting resistor of 220 Ohms. When SW1 is pressed pin 2 is pulled to ground causing output to go high (pin 3)."
- note added: "Pin 4 (Reset) is connected to Vcc to prevent accidently resets."
- note added: "Pin 5 (CV/Control) is grounded with a capacitor so that it does not consume much power and does not change the default operation of the 555 timer. This pin controls the threshold and trigger voltages and it is set to 2/3Vdd. The capacitor will help maintain this voltage consitently."
- note added: "R2 and C2 for our timing circuit. When pin 2 gets pulled to ground DIS becomes an open drain (not connected to Vcc or GND) which allows C2 to charge through R2. Once the threshold (pin 6) reaches the threshold voltage output (pin 3) will go low and the discharge pin will also go low causing the capacitor to quickly discharge. On page 15 of this datasheet, https://www.ti.com/lit/ds/symlink/tlc555.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"
- note added: "t=1.1*R*C=1.1*(10Mohm)(3.3uF) = 36.3s Will not be exactly that since the capacitor is rated to within 20% of its value and the resistor is within 5% of its value. A more accurate resistor and capacitor would make a more accurate timer. The 555 is most definitely the most accurate component here."
- note removed: "V=IR V=Vcc - Vled = 3V - 2V = 1V R=V/I = 1V/10mA = 100ohms I and Vled are take from this particular LED: https://www.digikey.ca/en/products/detail/sunled/XLUG11D/4745837 Use 220 ohm values for now."
- note removed: "t=RC=(10Mohm)(3.3uF) = 33s"
Changed lines of the file:
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@@
     (stroke (width 0) (type default) (color 0 0 0 0))
   )
-  (text "t=RC=(10Mohm)(3.3uF) = 33s" (at 194.31 77.47 0)
+  (text "Pin 4 (Reset) is connected to Vcc to prevent accidently resets."
+    (at 26.67 82.55 0)
     (effects (font (size 1.27 1.27)) (justify left bottom))
   )
-  (text "V=IR\nV=Vcc - Vled = 3V - 2V = 1V\nR=V/I = 1V/10mA = 100ohms\n\nI and Vled are take from this\nparticular LED: https://www.digikey.ca/en/products/detail/sunled/XLUG11D/4745837\n\nUse 220 ohm values for now."
-    (at 91.44 143.51 0)
+  (text "t=1.1*R*C=1.1*(10Mohm)(3.3uF) = 36.3s\nWill not be exactly that since the capacitor is \nrated to within 20% of its value and the resistor\nis within 5% of its value. \nA more accurate resistor and capacitor would make\na more accurate timer. The 555 is most definitely \nthe most accurate component here."
+    (at 201.93 87.63 0)
+    (effects (font (size 1.27 1.27)) (justify left bottom))
+  )
+  (text "Pin 2 is pulled high with a current limiting resistor\nof 220 Ohms. When SW1 is pressed pin 2 is pulled to \nground causing output to go high (pin 3)."
+    (at 77.47 62.23 0)
+    (effects (font (size 1.27 1.27)) (justify left bottom))
+  )
+  (text "Pin 5 (CV/Control) is grounded with a capacitor\nso that it does not consume much power and does\nnot change the default operation of the 555 timer.\n\nThis pin controls the threshold and trigger voltages\nand it is set to 2/3Vdd. The capacitor will help\nmaintain this voltage consitently."
+    (at 26.67 99.06 0)
+    (effects (font (size 1.27 1.27)) (justify left bottom))
+  )
+  (text "Lets figure the off current.\nThe 10M Ohm resistor will have a current draw.\nVcc=IR -> 6V=I (10M Ohm)\n-> I = 6V/(10M Ohm) = 0.6uA (micro-amps!)\n\nNot very much there!\n\nOn page one of the data sheet we see P=1mW at Vdd = 5V\nlets figure out the current consumption:\nP=VI -> I = P/V -> I = 1mW/5V = 0.2mA.\n\nSo that is more significant! \n\nPlus our batteries discharge about 1% a year by\nthemselves (see energizier doc). \n\nIn one year our 555 timer will use aproximately\n1752mA, so our batteries would be drained. \n\nLet's figure how long it will last approximately\nI = 0.2mA\nPbatt = 470mAh = I*(time in hours)\n-> time = 470mAh/0.2mA = 2350 hours = 98 days\nSo approximately 3 months!\n\nShould be enough for easter season."
+    (at 223.52 153.67 0)
+    (effects (font (size 1.27 1.27)) (justify left bottom))
+  )
+  (text "Let's figure the approximate LED current.\nVcc = 6V (will be a bit less)\nVpled = forward voltage of the purple LED = 3.2V\nVrled = forward voltage of the red LED = 2V\nVoled = forward voltage of the orange LED = 2V\nR = 220 Ohm\n\nIrled = Ioled\nV=Vcc - Vrled=IR\nIrled = 4V/220 Ohm = 18mA\n\nIpled = 13 mA\n\nThere may be rounding errors in these calculations\nbut they should be fairly close.\nThis means that the total current consumption is\njust under 50mA when turned on. \n\nWe have two CR2032 batteries which have approximately\n235mAh, https://data.energizer.com/pdfs/cr2032.pdf,\nso that is 470mAh. Our little device should be \nable to last 9 hours on (1080 cycles). \nThis will vary based on how long you leave it not\non since a small amount of current will be used \nwhen off. Where do you think that current is?"
+    (at 100.33 179.07 0)
+    (effects (font (size 1.27 1.27)) (justify left bottom))
+  )
+  (text "R2 and C2 for our timing circuit. When pin 2 gets\npulled to ground DIS becomes an open drain (not \nconnected to Vcc or GND) which allows C2 to charge\nthrough R2. Once the threshold (pin 6) reaches the\nthreshold voltage output (pin 3) will go low and \nthe discharge pin will also go low causing the \ncapacitor to quickly discharge. On page 15 of this\ndatasheet, https://www.ti.com/lit/ds/symlink/tlc555.pdf,\nwe see the capacitor will take approximately (1.1)(C2)(R2)\nto reach the threshold voltage. In this project a large \nresistor is chosen in conjunction with a medium value \ncapacitor to create a 36s output time."
+    (at 203.2 67.31 0)
     (effects (font (size 1.27 1.27)) (justify left bottom))
   )
@@
     )
     (pin "1")
-  )
-  (symbol (lib_id "Device:C_Polarized") (at 135.89 76.2 270) (unit 1)
-    (in_bom yes) (on_board yes)
-    (property "Reference" "C1" (id 0) (at 132.08 80.01 90))
-    (property "Value" "0.1u" (id 1) (at 132.08 82.55 90))
-    (property "Footprint" "Capacitor_THT:CP_Radial_D4.0mm_P2.00mm" (id 2) (at 132.08 77.1652 0)
-      (effects (font (size 1.27 1.27)) hide)
-    )
-    (property "Datasheet" "~" (id 3) (at 135.89 76.2 0)
-      (effects (font (size 1.27 1.27)) hide)
-    )
-    (pin "1")
-    (pin "2")
   )
   (symbol (lib_id "power:GND") (at 124.46 121.92 90) (unit 1)
@@
     (pin "2")
   )
+  (symbol (lib_id "Device:C") (at 135.89 76.2 270) (unit 1)
+    (in_bom yes) (on_board yes)
+    (property "Reference" "C1" (id 0) (at 135.89 80.01 90))
+    (property "Value" "0.1U" (id 1) (at 135.89 82.55 90))
+    (property "Footprint" "Capacitor_THT:CP_Radial_D5.0mm_P2.50mm" (id 2) (at 132.08 77.1652 0)
+      (effects (font (size 1.27 1.27)) hide)
+    )
+    (property "Datasheet" "~" (id 3) (at 135.89 76.2 0)
+      (effects (font (size 1.27 1.27)) hide)
+    )
+    (pin "1")
+    (pin "2")
+  )
   (symbol (lib_id "power:VCC") (at 190.5 55.88 0) (unit 1)
     (in_bom yes) (on_board yes) (fields_autoplaced)
@@
       (reference "BT2") (unit 1) (value "3v") (footprint "footprints:1066")
     )
-    (path "/1753b1a2-ed2d-4252-9dd8-88a2cffc6cef"
-      (reference "C1") (unit 1) (value "0.1u") (footprint "Capacitor_THT:CP_Radial_D4.0mm_P2.00mm")
+    (path "/da4bc8e5-66d4-4b93-9ddb-8b6cc82428a6"
+      (reference "C1") (unit 1) (value "0.1U") (footprint "Capacitor_THT:CP_Radial_D5.0mm_P2.50mm")
     )
     (path "/9a449d49-73da-49cd-8f8c-5056051c33a9"
